Commit message: Update to gazebo harmonic.

File: urdf/atreus.gazebo.xacro (robot description, xacro)
@@ -2,37 +2,40 @@
 <robot xmlns:xacro="http://www.ros.org/wiki/xacro" name="atreus">
 <gazebo>
-  <static>false</static>
+    <plugin filename="gz-sim-sensors-system" name="gz::sim::systems::Sensors">
+        <render_engine>ogre2</render_engine>
+    </plugin>
+    <plugin filename="gz-sim-imu-system" name="gz::sim::systems::Imu">
+    </plugin>
+    <plugin filename="gz-sim-joint-state-publisher-system" name="gz::sim::systems::JointStatePublisher">
+    </plugin>
 </gazebo>
-<!-- ..................... SKID-STEER DRIVE ........................................... -->
+<!-- ..................... MECANUM DRIVE ........................................... -->
 <gazebo>
-	<plugin name='skid_steer_drive' filename='libgazebo_ros_diff_drive.so'>
-    <ros>
-      <namespace>/</namespace>
-      <remapping>cmd_vel:=cmd_vel</remapping>
-      <remapping>odom:=odom</remapping>
-    </ros>
-    <!-- Number of wheel pairs -->
-    <num_wheel_pairs>2</num_wheel_pairs>
-    <!-- back wheels -->
-    <left_joint>back_left_wheel_joint</left_joint>
-    <right_joint>back_right_wheel_joint</right_joint>
-    <!-- front wheels-->
-    <left_joint>front_left_wheel_joint</left_joint>
-    <right_joint>front_right_wheel_joint</right_joint>
-    <!-- kinematics -->
-    <wheel_separation>${wheel_base}</wheel_separation>
-    <wheel_separation>${wheel_base}</wheel_separation>
-    <wheel_diameter>${2*wheel_radius}</wheel_diameter>
-    <wheel_diameter>${2*wheel_radius}</wheel_diameter>
-    <!-- limits -->
-    <max_wheel_torque>${wheel_torque}</max_wheel_torque>
-    <max_wheel_acceleration>0</max_wheel_acceleration>
-    <!-- output -->
-    <publish_odom>true</publish_odom>
-    <publish_odom_tf>true</publish_odom_tf>
-    <publish_wheel_tf>true</publish_wheel_tf>
-    <odometry_frame>odom</odometry_frame>
-    <robot_base_frame>base_link</robot_base_frame>
-    <update_rate>50</update_rate>
+  <plugin filename="gz-sim-mecanum-drive-system" name="gz::sim::systems::MecanumDrive">
+    <front_left_joint>front_left_wheel_joint</front_left_joint>
+    <front_right_joint>front_right_wheel_joint</front_right_joint>
+    <back_left_joint>back_left_wheel_joint</back_left_joint>
+    <back_right_joint>back_right_wheel_joint</back_right_joint>
+    <wheelbase>${wheel_base}</wheelbase>
+    <wheel_separation>${wheel_separation}</wheel_separation>
+    <wheel_radius>${wheel_radius}</wheel_radius>
+    <odom_publish_frequency>30</odom_publish_frequency>
+    <topic>cmd_vel</topic>
+    <odom_topic>encoder_odom</odom_topic>
+    <tf_topic>/tf</tf_topic>
+    <frame_id>odom</frame_id>
+    <child_frame_id>base_link</child_frame_id>
+  </plugin>
+</gazebo>
+<!-- ............................. GAZEBO ODOM .................................... -->
+<gazebo>
+    <plugin filename="libgz-sim-odometry-publisher-system"
+        name="gz::sim::systems::OdometryPublisher">
+        <odom_frame>odom</odom_frame>
+        <robot_base_frame>base_link</robot_base_frame>
+        <odom_topic>gazebo_odom</odom_topic>
+        <tf_topic>/tf</tf_topic>
+        <dimensions>2</dimensions>
+        <odom_publish_frequency>10</odom_publish_frequency>
     </plugin>
 </gazebo>
@@ -45,72 +48,9 @@
 <gazebo reference="imu_link">
   <sensor name="imu_sensor" type="imu">
-    <always_on>true</always_on>
-    <!-- Publish at 30 hz -->
-    <update_rate>30</update_rate>
-    <!-- frame_name omitted, will be "imu_link" -->
-    <frame_name>imu_link</frame_name> <!-- Redundant -->
-    <!-- Custom Gazebo noise -->
-    <imu>
-      <angular_velocity>
-        <x>
-          <noise type="gaussian">
-            <mean>0</mean>
-            <stddev>0.0002</stddev>
-            <bias_mean>7.5e-06</bias_mean>
-            <bias_stddev>8e-07</bias_stddev>
-          </noise>
-        </x>
-        <y>
-          <noise type="gaussian">
-            <mean>0</mean>
-            <stddev>0.0002</stddev>
-            <bias_mean>7.5e-06</bias_mean>
-            <bias_stddev>8e-07</bias_stddev>
-          </noise>
-        </y>
-        <z>
-          <noise type="gaussian">
-            <mean>0</mean>
-            <stddev>0.0002</stddev>
-            <bias_mean>7.5e-06</bias_mean>
-            <bias_stddev>8e-07</bias_stddev>
-          </noise>
-        </z>
-      </angular_velocity>
-      <linear_acceleration>
-        <x>
-          <noise type="gaussian">
-            <mean>0</mean>
-            <stddev>0.017</stddev>
-            <bias_mean>0.1</bias_mean>
-            <bias_stddev>0.001</bias_stddev>
-          </noise>
-        </x>
-        <y>
-          <noise type="gaussian">
-            <mean>0</mean>
-            <stddev>0.017</stddev>
-            <bias_mean>0.1</bias_mean>
-            <bias_stddev>0.001</bias_stddev>
-          </noise>
-        </y>
-        <z>
-          <noise type="gaussian">
-            <mean>0</mean>
-            <stddev>0.017</stddev>
-            <bias_mean>0.1</bias_mean>
-            <bias_stddev>0.001</bias_stddev>
-          </noise>
-        </z>
-      </linear_acceleration>
-    </imu>
-    <plugin name="imu_plugin" filename="libgazebo_ros_imu_sensor.so">
-      <ros>
-        <!-- Will publish to /imu/data -->
-        <namespace>/imu</namespace>
-        <remapping>~/out:=data</remapping> <!-- Don't use arguments, as the updated version is buggy-->
-      </ros>
-      <initial_orientation_as_reference>false</initial_orientation_as_reference>
-    </plugin>
+      <always_on>1</always_on>
+      <update_rate>1</update_rate>
+      <visualize>true</visualize>
+      <topic>imu</topic>
+      <ignition_frame_id>imu_frame</ignition_frame_id>
   </sensor>
 </gazebo>
@@ -118,52 +58,21 @@
 <xacro:if value="$(arg camera_enabled)">
   <gazebo reference="camera_link">
-    <sensor type="camera" name="camera">
-      <!-- Set always_on only sensor, not on plugin -->
-      <always_on>0</always_on>
-      <!-- Set update_rate only sensor, not on plugin -->
-      <update_rate>30</update_rate>
-      <camera name="front_camera">
-          <horizontal_fov>${radians(camera_horizontal_fov)}</horizontal_fov>
-          <image>
-              <width>640</width>
-              <height>480</height>
-              <format>RGB_INT8</format>
-          </image>
-          <clip>
-              <near>0.1</near>
-              <far>10</far>
-          </clip>
-          <noise>
-            <type>gaussian</type>
-            <mean>0.0</mean>
-            <stddev>0.007</stddev>
-          </noise>
-        <distortion>
-          <k1>0.0</k1>
-          <k2>0.0</k2>
-          <k3>0.0</k3>
-          <p1>0.0</p1>
-          <p2>0.0</p2>
-          <center>0.0 0.0</center>
-        </distortion>
-      </camera>
-      <!-- Use camera, not camera_triggered -->
-      <plugin name="plugin_name" filename="libgazebo_ros_camera.so">
-        <!-- DON'T USE COLON-->
-        <!-- Change namespace, camera name and topics so -
-              * Images are published to- /custom_ns/custom_camera/custom_image
-              * Camera info is published to- /custom_ns/custom_camera/custom_info  -->
-        <ros>
-          <namespace></namespace>
-          <remapping>image_raw:=image_raw</remapping>
-          <remapping>camera_info:=camera_info</remapping>
-        </ros>
-        <!-- Set camera name. If empty, defaults to sensor name (i.e. "sensor_name") -->
-        <camera_name>camera</camera_name>
-        <!-- Set TF frame name. If empty, defaults to link name (i.e. "link_name") -->
-        <frame_name>camera_link</frame_name>
-        <hack_baseline>0.07</hack_baseline>
-        <!-- No need to repeat distortion parameters or to set autoDistortion -->
-      </plugin>
+    <sensor type="depth_camera" name="kinect_camera">
+        <update_rate>30.0</update_rate>
+        <topic>camera</topic>
+        <gz_frame_id>camera_link</gz_frame_id>
+        <camera>
+            <camera_info_topic>camera_info</camera_info_topic>
+            <horizontal_fov>${radians(camera_horizontal_fov)}</horizontal_fov>
+            <image>
+                <width>640</width>
+                <height>480</height>
+                <format>R8G8B8</format>
+            </image>
+            <clip>
+                <near>0.05</near>
+                <far>8.0</far>
+            </clip>
+        </camera>
     </sensor>
   </gazebo>
@@ -171,38 +80,33 @@
 <!-- ........................... 2D LIDAR PLUGIN ................................... -->
 <xacro:if value="$(arg two_d_lidar_enabled)">
-   <gazebo reference="two_d_lidar">
-    <sensor type="ray" name="lidar_sensor">
-      <ray>
-        <scan>
-          <horizontal>
-            <samples>${two_d_lidar_sample_size}</samples>
-            <resolution>1</resolution>
-            <min_angle>${radians(two_d_lidar_min_angle)}</min_angle>
-            <max_angle>${radians(two_d_lidar_max_angle)}</max_angle>
-          </horizontal>
-        </scan>
-        <range>
-          <min>${two_d_lidar_min_range}</min>
-          <max>${two_d_lidar_max_range}</max>
-          <resolution>0.01</resolution>
-        </range>
-        <noise>
-          <type>gaussian</type>
-          <mean>0.0</mean>
-          <stddev>0.001</stddev>
-        </noise>
-      </ray>
-      <update_rate>${two_d_lidar_update_rate}</update_rate>
-      <visualize>false</visualize>
-      <plugin name="gazebo_ros_laser" filename="libgazebo_ros_ray_sensor.so">
-        <ros>
-          <namespace>/</namespace>
-          <remapping>~/out:=scan</remapping>
-        </ros>
-        <output_type>sensor_msgs/LaserScan</output_type>
-        <frame_name>two_d_lidar</frame_name>
-      </plugin>
-    </sensor>
-   </gazebo>
+  <gazebo reference="two_d_lidar">
+      <sensor name='gpu_lidar' type='gpu_lidar'>
+          <topic>scan</topic>
+          <update_rate>${two_d_lidar_update_rate}</update_rate>
+          <gz_frame_id>two_d_lidar</gz_frame_id>
+          <lidar>
+              <scan>
+                  <horizontal>
+                      <samples>${two_d_lidar_sample_size}</samples>
+                      <resolution>1</resolution>
+                      <min_angle>${radians(two_d_lidar_min_angle)}</min_angle>
+                      <max_angle>${radians(two_d_lidar_max_angle)}</max_angle>
+                  </horizontal>
+              </scan>
+              <range>
+                  <min>${two_d_lidar_min_range}</min>
+                  <max>${two_d_lidar_max_range}</max>
+                  <resolution>0.01</resolution>
+              </range>
+              <noise>
+                  <type>gaussian</type>
+                  <mean>0.0</mean>
+                  <stddev>0.001</stddev>
+              </noise>
+          </lidar>
+          <always_on>1</always_on>
+          <visualize>true</visualize>
+      </sensor>
+  </gazebo>
 </xacro:if>
 <!--................................................................................. -->

File: urdf/atreus.xacro (robot description, xacro)
@@ -24,5 +24,6 @@
 <!-- Z distance to centre of the robot -->
 <xacro:property name="chassis_ground_clearance"             value="${0.1+chassis_height/2}"/>
-<xacro:property name="wheel_base"                           value="${wheel_width+chassis_width}"/>
+<xacro:property name="wheel_base"                           value="${wheel_pos-chassis_length/4+wheel_radius}"/>
+<xacro:property name="wheel_separation"                     value="${wheel_width+chassis_width}"/>
 <!-- ............................... LOAD MACROS ................................. -->
 <xacro:include filename="$(find atreus)/urdf/atreus.gazebo.xacro"/>
@@ -87,5 +88,5 @@
       <material>Gazebo/Purple</material>
   </gazebo>
-  <!-- CAMERA -->
+  <!-- 3D CAMERA -->
     <link name="camera_link">
       <collision>

File: urdf/macros.xacro (robot description, xacro)
@@ -45,5 +45,5 @@
       <parent link="base_link"/>
       <child link="${cardinality}_${dexterity}_wheel"/>
-      <origin xyz="${fb*(wheel_pos-chassis_length/4+wheel_radius)} ${lr*(wheel_width/2+chassis_width/2)} ${wheel_radius}" rpy="0 0 0" />
+      <origin xyz="${fb*(wheel_base)} ${lr*(wheel_separation/2)} ${wheel_radius}" rpy="0 0 0" />
       <axis xyz="0 1 0" rpy="0 0 0" />
     </joint>
